File: PCB/v0.2/TeensyROM.brd (EAGLE design)
At the start: 61 x 56.6 mm, 23 parts, among them J1 C64-EXPANSION-PORT, J2 3 pin Header, U1 TEENSY41, U2 74LCV245, U3 74LCV245, U4 74LCV245, U5 74LCV245, U6 74LVC07, X2 SI-50170

Commit message: PCB 0.2 progress (not yet complete)
Parts:
- removed X2: SI-50170, TeensyROM:SI-50170
- added J3: J1B1211CCD, TeensyROM:CONN12_J1B1211CCD_WIZ
- added S1: SHORTSMT, AudioLooper:SHORT
- C9: value (none) -> 100uF
- moved C9 25.1 mm to (33.4, 63.0), flipped to the bottom
- moved C8 21.7 mm to (15.1, 52.1), flipped to the bottom
- moved C2 9.46 mm to (20.1, 54.7)
- moved C1 9.42 mm to (20.1, 60.7)
- moved X1 9.06 mm to (31.5, 70.0)
- moved D1 4.07 mm to (47.2, 65.2)
- moved B1 3.42 mm to (54.5, 64.2)
- moved R1 1.42 mm to (55.5, 58.9), flipped to the bottom
- moved U1 1.27 mm to (30.5, 40.6)
- moved C3 1.14 mm to (3.81, 20.1), turned to 90 degrees
- moved C5 1.14 mm to (31.2, 20.8), turned to 270 degrees
- moved J2 1.05 mm to (55.1, 51.6), turned to 180 degrees
- moved R2 0.51 mm to (52.3, 57.1), flipped to the bottom, turned to 270 degrees
Connections:
- net N$1 renamed LED_R
- removed net N$2: C8.2, X2.2, X2.5
- new net ETH_CT: C8.2, J3.2, J3.5
- new net ETH_SH: J3.S1, J3.S2, S1.2
- net +3V3: no longer U1.3V3-2
- net DM: now also X1.D-
- net DP: now also X1.D+
- net ETH_LED: now also J3.10; no longer X2.A1
- net ETH_R+: now also J3.4; no longer X2.4
- net ETH_R-: now also J3.6; no longer X2.6
- net ETH_T+: now also J3.1; no longer X2.1
- net ETH_T-: now also J3.3; no longer X2.3
- net GND: now also J3.11, J3.8, J3.9, S1.1, X1.SH2; no longer U1.GND2, X2.8, X2.C1
- net VHST: now also U1.+5V, X1.5V; no longer U1.VUSB
Routing:
- net VHST: track 0.00 -> 44.6 mm
- net DP: track 0.00 -> 37.8 mm
- net DM: track 0.00 -> 37.7 mm
- net GND: track 373.0 -> 339.5 mm, vias 13 -> 12
- net +3V3: track 203.1 -> 172.1 mm, vias 6 -> 7
- net ETH_LED: track 0.00 -> 28.4 mm
- net ETH_T-: track 0.00 -> 18.1 mm
- net ETH_T+: track 0.00 -> 18.0 mm
- net ETH_SH: track 0.00 -> 17.3 mm
- net ETH_R-: track 0.00 -> 13.9 mm
- net ETH_R+: track 0.00 -> 13.9 mm
- net !BUTTON: track 17.0 -> 30.3 mm
- net ETH_CT: track 0.00 -> 12.5 mm
- net LED: track 1.27 -> 6.01 mm
- net A7_B: track 39.7 -> 43.5 mm
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Other:
- board size 61 x 56.6 mm -> 61 x 68.6 mm
- board text added: "Top Side"
- board text added: "v0.2"
- board text removed: "v0.1"
