File: PCB/v0.2 archive/TeensyROM.brd (EAGLE design)
At the start: 61 x 68.6 mm, 24 parts, among them J1 C64-EXPANSION-PORT, J2 292303-1, J3 J1B1211CCD, J4 3 pin Header, U1 TEENSY41, U2 74LCV245, U3 74LCV245, U4 74LCV245, U5 74LCV245, U6 74LVC07

Commit message: Minor rev to PCB 0.2 (now 0.2b) to include pull-up on Data_CE
Parts:
- added R3: 10k, resistor:R0805
Connections:
- net !DATA_CE: now also R3.2
- net +3V3: now also R3.1
Routing:
- net +3V3: track 207.9 -> 212.1 mm
- net !DATA_CE: track 42.5 -> 46.6 mm
Other:
- board text added: "v0.2b"
- board text removed: "v0.2"
Changed lines of the file:
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@@
 <wire x1="57.1881" y1="0" x2="58.0136" y2="0.8255" width="0" layer="20" curve="90"/>
 <wire x1="0" y1="-2.54" x2="58.166" y2="-2.54" width="0.4064" layer="51"/>
-<text x="46.3042" y="49.9872" size="2.286" layer="21" font="vector" ratio="12">v0.2</text>
+<text x="46.3042" y="49.9872" size="2.286" layer="21" font="vector" ratio="12">v0.2b</text>
 <text x="1.778" y="27.813" size="1.651" layer="21" font="vector" ratio="13">github.com/SensoriumEmbedded/TeensyROM</text>
 <text x="23.0378" y="52.832" size="4.064" layer="21" font="vector" ratio="15">TeensyROM</text>
@@
 <attribute name="VALUE" x="16.256" y="60.96" size="1.27" layer="28" rot="MR270"/>
 </element>
+<element name="R3" library="resistor" package="R0805" value="10k" x="53.34" y="53.34" smashed="yes" rot="MR270">
+<attribute name="NAME" x="50.165" y="53.975" size="1.143" layer="26" font="vector" ratio="10" rot="MR180"/>
+<attribute name="VALUE" x="55.88" y="53.975" size="1.27" layer="28" rot="MR270"/>
+</element>
 </elements>
 <signals>
@@
 <wire x1="17.642" y1="18.277" x2="17.78" y2="18.415" width="0.6096" layer="16"/>
 <wire x1="46.355" y1="37.211" x2="45.085" y2="37.211" width="1.27" layer="1"/>
-<wire x1="54.229" y1="57.978" x2="51.877" y2="57.978" width="0.1524" layer="16"/>
-<wire x1="51.877" y1="57.978" x2="50.8" y2="59.055" width="0.1524" layer="16"/>
 <via x="50.8" y="59.055" extent="1-16" drill="0.6"/>
 <wire x1="50.8" y1="59.055" x2="48.895" y2="59.055" width="0.1524" layer="1"/>
@@
 <wire x1="3.556" y1="20.839" x2="3.556" y2="21.971" width="0.6096" layer="1"/>
 <wire x1="3.556" y1="21.971" x2="3.81" y2="22.225" width="0.6096" layer="1"/>
+<contactref element="R3" pad="1"/>
+<wire x1="53.34" y1="54.29" x2="53.34" y2="56.515" width="0.254" layer="16"/>
+<wire x1="53.34" y1="56.515" x2="50.8" y2="59.055" width="0.254" layer="16"/>
+<wire x1="54.229" y1="57.978" x2="54.229" y2="56.769" width="0.254" layer="16"/>
+<wire x1="54.229" y1="56.769" x2="53.975" y2="56.515" width="0.254" layer="16"/>
+<wire x1="53.975" y1="56.515" x2="53.34" y2="56.515" width="0.254" layer="16"/>
 </signal>
 <signal name="A15_B">
@@
 <wire x1="51.054" y1="12.446" x2="50.8" y2="12.7" width="0.1524" layer="1"/>
 <wire x1="50.8" y1="12.7" x2="50.8" y2="14.2748" width="0.1524" layer="1"/>
+<contactref element="R3" pad="2"/>
+<wire x1="53.34" y1="52.39" x2="53.34" y2="48.26" width="0.1524" layer="16"/>
 </signal>
 <signal name="A7_B">

Commit message: R1 val change, PDF update
Parts:
- R1: value 1k -> 10k
Changed lines of the file:
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@@
 <attribute name="VALUE" x="60.96" y="51.181" size="1.27" layer="27" rot="R90"/>
 </element>
-<element name="R1" library="resistor" package="R0805" value="1k" x="54.229" y="58.928" smashed="yes" rot="MR270">
+<element name="R1" library="resistor" package="R0805" value="10k" x="54.229" y="58.928" smashed="yes" rot="MR270">
 <attribute name="NAME" x="51.0794" y="59.4868" size="1.143" layer="26" font="vector" ratio="10" rot="MR180"/>
 <attribute name="VALUE" x="56.769" y="59.563" size="1.27" layer="28" rot="MR270"/>
