File: PCB/v0.2 archive/TeensyROM.sch (EAGLE design)
At the start: 24 parts, among them J1 C64-EXPANSION-PORT, J2 292303-1, J3 J1B1211CCD, J4 3 pin Header, U1 TEENSY41, U2 74LCV245, U3 74LCV245, U4 74LCV245, U5 74LCV245, U6 74LVC07

Commit message: Minor rev to PCB 0.2 (now 0.2b) to include pull-up on Data_CE
Parts:
- added R3: 10k, resistor:R-US_R0805
Connections:
- net !DATA_CE: now also R3.2
- net +3V3: now also R3.1
Other:
- note added: "0.2b"
- note removed: "0.2"
- moved on the sheet: C7, U5

Commit message: R1 val change, PDF update
Parts:
- R1: value 1k -> 10k
Changed lines of the file:
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@@
 <part name="SUPPLY3" library="supply2" deviceset="GND" device=""/>
 <part name="J4" library="TeensyROM" deviceset="PINHD-1X3" device="" value="3 pin Header"/>
-<part name="R1" library="resistor" deviceset="R-US_" device="R0805" value="1k"/>
+<part name="R1" library="resistor" deviceset="R-US_" device="R0805" value="10k"/>
 <part name="SUPPLY13" library="supply2" deviceset="GND" device=""/>
 <part name="+3V7" library="supply1" deviceset="+3V3" device=""/>
